File: FC_ESP32/FC_ESP32.kicad_pcb (KiCad board)
At the start: 2 copper layers, 79.8 x 79.8 mm, 76 parts, among them J1 USB4105-GF-A, J2 MTF-01P SH1.0, J3 BAT 1S, J4 M1 + / -, J5 M2 + / -, J6 M3 + / -, J7 M4 + / -, J8 I2C, J9 UART1, Q1 AO3400, Q2 AO3400, Q3 AO3400, Q4 AO3400, Q5 MMBT3904, Q6 MMBT3904, U1 ESP32-WROOM-32 (8MB), U2 MPU-6500, U3 CH340C, U4 USBLC6-2SC6, U5 TPS63001DRCR, U6 TPS61070DDCR

Commit message: .
Routing:
- net +5V_FLOW: track 0.00 -> 82.0 mm, vias 0 -> 10
- net EN: track 92.1 -> 102.2 mm, vias 9 -> 11
