File: FC_ESP32/FC_ESP32.kicad_sch (KiCad schematic)
At the start: 0 parts

Commit message: .
Parts:
- added C1, C17: 22uF 10V X5R, FC_Local:C_0805_2012Metric, symbol FC_Local:C
- added C11: 1uF 10V, FC_Local:C_0603_1608Metric, symbol FC_Local:C
- added C12, C13: 10uF 10V X5R, FC_Local:C_0805_2012Metric, symbol FC_Local:C
- added C15, C18, C2, C4, C5, C7, C9: 100nF, FC_Local:C_0402_1005Metric, symbol FC_Local:C
- added C19: 47uF 10V X5R, FC_Local:C_1206_3216Metric, symbol FC_Local:C
- added C21, C22, C23, C24: 100nF 10V, FC_Local:C_0603_1608Metric, symbol FC_Local:C
- added C3: 1uF, FC_Local:C_0603_1608Metric, symbol FC_Local:C
- added C6: 10nF, FC_Local:C_0402_1005Metric, symbol FC_Local:C
- added C8: 1uF, FC_Local:C_0402_1005Metric, symbol FC_Local:C
- added D1, D2, D3, D4, D5, D6: SS16, FC_Local:SS16, symbol FC_Local:SS16
- added J1: USB4105-GF-A, FC_Local:USB_C, symbol FC_Local:USB_C
- added J2: MTF-01P SH1.0, FC_Local:JST_SH_SM04B-SRSS-TB_1x04-1MP_P1.00mm_Horizontal, symbol FC_Local:Conn4
- added J3: BAT 1S, FC_Local:Battery_Wire_Pads, symbol FC_Local:Conn2
- added J4: M1 + / -, FC_Local:Motor_Wire_Pads, symbol FC_Local:Conn2
- added J5: M2 + / -, FC_Local:Motor_Wire_Pads, symbol FC_Local:Conn2
- added J6: M3 + / -, FC_Local:Motor_Wire_Pads, symbol FC_Local:Conn2
- added J7: M4 + / -, FC_Local:Motor_Wire_Pads, symbol FC_Local:Conn2
- added J8: I2C, FC_Local:Header_1x04_P2.54mm, symbol FC_Local:Conn4
- added J9: UART1, FC_Local:Header_1x04_P2.54mm, symbol FC_Local:Conn4
- added L1: 2.2uH VLF4012-2R2M1R5, FC_Local:L_VLF4012, symbol FC_Local:L
- added L2: 4.7uH >=1A shielded, FC_Local:L_4x4, symbol FC_Local:L
- added Q1, Q2, Q3, Q4: AO3400, FC_Local:AO3400, symbol FC_Local:AO3400
- added Q5, Q6: MMBT3904, FC_Local:MMBT3904, symbol FC_Local:MMBT3904
- added R1, R10, R2, R6, R9: 10k, FC_Local:R_0402_1005Metric, symbol FC_Local:R
- added R11, R15, R17, R19, R21: 100R, FC_Local:R_0402_1005Metric, symbol FC_Local:R
- added R12: 1.8M 1%, FC_Local:R_0402_1005Metric, symbol FC_Local:R
- added R13: 200k 1%, FC_Local:R_0402_1005Metric, symbol FC_Local:R
- added R16, R18, R20, R22: 100k, FC_Local:R_0402_1005Metric, symbol FC_Local:R
- added R23, R24: 4.7k, FC_Local:R_0402_1005Metric, symbol FC_Local:R
- added R3, R4: 100k 1%, FC_Local:R_0402_1005Metric, symbol FC_Local:R
- added R5: 10R, FC_Local:R_0402_1005Metric, symbol FC_Local:R
- added R7, R8: 5.1k 1%, FC_Local:R_0402_1005Metric, symbol FC_Local:R
- added U1: ESP32-WROOM-32 (8MB), FC_Local:ESP32, symbol FC_Local:ESP32
- added U2: MPU-6500, FC_Local:MPU6500, symbol FC_Local:MPU6500
- added U3: CH340C, FC_Local:CH340C, symbol FC_Local:CH340C
- added U4: USBLC6-2SC6, FC_Local:SOT-23-6, symbol FC_Local:USBLC6
- added U5: TPS63001DRCR, FC_Local:Texas_DRC0010J, symbol FC_Local:TPS63001
- added U6: TPS61070DDCR, FC_Local:SOT-23-6, symbol FC_Local:TPS61070
Connections:
- new net +3V3: C1.1, C13.1, C2.1, C9.1, J8.1 (Pin_1), J9.1 (Pin_1), L2.1, R1.1, R2.1, R23.1, R24.1, R5.1, U1.2 (3V3), U3.16 (VCC), U3.4 (V3), U5.1 (VOUT), U5.10 (FB), U6.3 (EN), U6.6 (VBAT)
- new net +3V3_IMU: C5.1, C6.1, C8.1, R5.2, R6.1, U2.13 (VDD), U2.8 (VDDIO)
- new net +5V_FLOW: C17.1, C18.1, J2.2 (Pin_2), R12.1, U6.5 (VOUT)
- new net BASE_BOOT: Q6.1, R10.2
- new net BASE_EN: Q5.1, R9.2
- new net BOOST_FB: R12.2, R13.1, U6.4 (FB)
- new net BOOST_SW: L2.2, U6.1 (SW)
- new net BOOT: Q6.3, R2.2, U1.25 (IO0)
- new net BUCK_L1: L1.1, U5.4 (L1)
- new net BUCK_L2: L1.2, U5.2 (L2)
- new net CC1: J1.A5 (CC1), R7.1
- new net CC2: J1.B5 (CC2), R8.1
- new net DTR: Q6.2, R9.1, U3.13 (~{DTR})
- new net EN: C3.1, Q5.3, R1.2, U1.3 (EN)
- new net FLOW_RX: J2.4 (Pin_4), U1.27 (IO16)
- new net FLOW_TX: J2.3 (Pin_3), U1.28 (IO17)
- new net GATE1: Q1.1, R15.2, R16.1
- new net GATE2: Q2.1, R17.2, R18.1
- new net GATE3: Q3.1, R19.2, R20.1
- new net GATE4: Q4.1, R21.2, R22.1
- new net GND: C1.2, C11.2, C12.2, C13.2, C15.2, C17.2, C18.2, C19.2, C2.2, C3.2, C4.2, C5.2, C6.2, C7.2, C8.2, C9.2, J1.A1 (GND), J1.A12 (GND), J1.B1 (GND), J1.B12 (GND), J1.SH (SHIELD), J2.1 (Pin_1), J3.2 (Pin_2), J8.2 (Pin_2), J9.2 (Pin_2), Q1.2, Q2.2, Q3.2, Q4.2, R13.2, R16.2, R18.2, R20.2, R22.2, R4.2, R7.2, R8.2, U1.1 (GND), U1.15 (GND), U1.38 (GND), U1.39 (GND), U2.11 (FSYNC), U2.18 (GND), U2.20 (RESV_2), U2.25 (EXP), U3.1 (GND), U3.15 (R232), U4.2 (GND), U5.11 (PGND), U5.3 (PGND), U5.9 (GND), U6.2 (GND)
- new net I2C_SCL: J8.4 (Pin_4), R24.2, U1.36 (IO22)
- new net I2C_SDA: J8.3 (Pin_3), R23.2, U1.26 (IO4)
- new net IMU_CS: R6.2, U1.33 (IO21), U2.22 (NCS)
- new net IMU_INT: U1.6 (IO34), U2.12 (INT)
- new net M1_NEG: C21.2, D1.2, J4.2 (Pin_2), Q1.3
- new net M2_NEG: C22.2, D2.2, J5.2 (Pin_2), Q2.3
- new net M3_NEG: C23.2, D3.2, J6.2 (Pin_2), Q3.3
- new net M4_NEG: C24.2, D4.2, J7.2 (Pin_2), Q4.3
- new net PWM1: R15.1, U1.10 (IO25)
- new net PWM2: R17.1, U1.11 (IO26)
- new net PWM3: R19.1, U1.12 (IO27)
- new net PWM4: R21.1, U1.9 (IO33)
- new net REGOUT: C7.1, U2.10 (REGOUT)
- new net RTS: Q5.2, R10.1, U3.14 (~{RTS})
- new net SPI_MISO: U1.31 (IO19), U2.9 (AD0/SDO)
- new net SPI_MOSI: U1.37 (IO23), U2.24 (SDA/SDI)
- new net SPI_SCK: U1.30 (IO18), U2.23 (SCL/SCLK)
- new net UART0_RX: U1.34 (RXD0), U3.2 (TXD)
- new net UART0_TX: U1.35 (TXD0), U3.3 (RXD)
- new net UART1_RX: J9.4 (Pin_4), U1.8 (IO32)
- new net UART1_TX: J9.3 (Pin_3), U1.13 (IO14)
- new net USB_DM: J1.A7 (D-), J1.B7 (D-), U3.6 (UD-), U4.1 (I/O1), U4.6 (I/O1)
- new net USB_DP: J1.A6 (D+), J1.B6 (D+), U3.5 (UD+), U4.3 (I/O2), U4.4 (I/O2)
- new net VBAT: C19.1, C21.1, C22.1, C23.1, C24.1, D1.1, D2.1, D3.1, D4.1, D5.2, J3.1 (Pin_1), J4.1 (Pin_1), J5.1 (Pin_1), J6.1 (Pin_1), J7.1 (Pin_1), R3.1
- new net VBAT_ADC: C4.1, R3.2, R4.1, U1.7 (IO35)
- new net VBUS: C11.1, D6.2, J1.A4 (VBUS), J1.A9 (VBUS), J1.B4 (VBUS), J1.B9 (VBUS), U4.5 (VBUS)
- new net VINA: C15.1, R11.2, U5.8 (VINA)
- new net VSYS: C12.1, D5.1, D6.1, R11.1, U5.5 (VIN), U5.6 (EN), U5.7 (PS/SYNC)
- no-connect marks 0 -> 24
Other:
- removed sheet 1S power distribution
- removed sheet ESP32 and battery measurement
- removed sheet Four brushed motor drivers
- removed sheet MPU6500 SPI and optical flow
- removed sheet USB-C programming and auto-reset
- note added: "IMU + FLOW (MPU6500 / J2)"
- note added: "MCU / BATTERY SENSE"
- note added: "MOTORS x4 (AO3400 + SS16)"
- note added: "POWER 1S (TPS63001 / TPS61070)"
- note added: "POWER RAILS"
- note added: "USB / CH340C + AUTO-RESET"
