File: validation/only_c3_ground_remaining.kicad_pcb (KiCad board)
At the start: 2 copper layers, 79.8 x 79.8 mm, 76 parts, among them J1 USB4105-GF-A, J2 MTF-01P SH1.0, J3 BAT 1S, J4 M1 + / -, J5 M2 + / -, J6 M3 + / -, J7 M4 + / -, J8 I2C, J9 UART1, Q1 AO3400, Q2 AO3400, Q3 AO3400, Q4 AO3400, Q5 MMBT3904, Q6 MMBT3904, U1 ESP32-WROOM-32 (8MB), U2 MPU-6500, U3 CH340C, U4 USBLC6-2SC6, U5 TPS63001DRCR, U6 TPS61070DDCR

Commit message: .
Routing:
- net BOOST_FB: track 0.00 -> 28.3 mm, vias 0 -> 5
Changed lines of the file:
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@@
+	)
+	(segment
+		(start 89.51 94.75)
+		(end 88.55 93.79)
+		(width 0.18)
+		(layer "F.Cu")
+		(net "BOOST_FB")
+	)
+	(segment
+		(start 87.0028 92.8112)
+		(end 86.5011 92.8112)
+		(width 0.18)
+		(layer "F.Cu")
+		(net "BOOST_FB")
+	)
+	(segment
+		(start 84.8625 89.55)
+		(end 83.8625 89.55)
+		(width 0.18)
+		(locked yes)
+		(layer "F.Cu")
+		(net "BOOST_FB")
+	)
+	(segment
+		(start 82.4762 82.653)
+		(end 81.4098 83.7194)
+		(width 0.18)
+		(layer "F.Cu")
+		(net "BOOST_FB")
+	)
+	(segment
+		(start 86.5011 92.8112)
+		(end 86.0149 92.325)
+		(width 0.18)
+		(layer "F.Cu")
+		(net "BOOST_FB")
+	)
+	(segment
+		(start 88.49 87)
+		(end 88.1051 87)
+		(width 0.18)
+		(layer "F.Cu")
+		(net "BOOST_FB")
+	)
+	(segment
+		(start 81.4098 85.5023)
+		(end 81.5346 85.6271)
+		(width 0.18)
+		(layer "F.Cu")
+		(net "BOOST_FB")
+	)
+	(segment
+		(start 88.55 93.79)
+		(end 88.55 92.8162)
+		(width 0.18)
+		(layer "F.Cu")
+		(net "BOOST_FB")
+	)
+	(segment
+		(start 88.55 92.8162)
+		(end 88.221 92.4872)
+		(width 0.18)
+		(layer "F.Cu")
+		(net "BOOST_FB")
+	)
+	(segment
+		(start 85.1539 89.55)
+		(end 86.0149 90.411)
+		(width 0.18)
+		(layer "F.Cu")
+		(net "BOOST_FB")
+	)
+	(segment
+		(start 87.3268 92.4872)
+		(end 87.0028 92.8112)
+		(width 0.18)
+		(layer "F.Cu")
+		(net "BOOST_FB")
+	)
+	(segment
+		(start 86.0149 90.411)
+		(end 86.0149 91.3515)
+		(width 0.18)
+		(layer "F.Cu")
+		(net "BOOST_FB")
+	)
+	(segment
+		(start 84.8625 89.55)
+		(end 85.1539 89.55)
+		(width 0.18)
+		(layer "F.Cu")
+		(net "BOOST_FB")
+	)
+	(segment
+		(start 86.0149 92.325)
+		(end 86.0149 91.3515)
+		(width 0.18)
+		(layer "F.Cu")
+		(net "BOOST_FB")
+	)
+	(segment
+		(start 88.221 92.4872)
+		(end 87.3268 92.4872)
+		(width 0.18)
+		(layer "F.Cu")
+		(net "BOOST_FB")
+	)
+	(segment
+		(start 88.1051 87)
+		(end 87.6367 86.5316)
+		(width 0.18)
+		(layer "F.Cu")
+		(net "BOOST_FB")
+	)
+	(segment
+		(start 81.4098 83.7194)
+		(end 81.4098 85.5023)
+		(width 0.18)
+		(layer "F.Cu")
+		(net "BOOST_FB")
+	)
+	(via
+		(at 83.8625 89.55)
+		(size 0.6)
+		(drill 0.3)
+		(layers "F.Cu" "B.Cu")
+		(locked yes)
+		(net "BOOST_FB")
+	)
+	(via
+		(at 81.5346 85.6271)
+		(size 0.6)
+		(drill 0.3)
+		(layers "F.Cu" "B.Cu")
+		(net "BOOST_FB")
+	)
+	(via
+		(at 82.4762 82.653)
+		(size 0.6)
+		(drill 0.3)
+		(layers "F.Cu" "B.Cu")
+		(net "BOOST_FB")
+	)
+	(via
+		(at 86.0149 91.3515)
+		(size 0.6)
+		(drill 0.3)
+		(layers "F.Cu" "B.Cu")
+		(net "BOOST_FB")
+	)
+	(via
+		(at 87.6367 86.5316)
+		(size 0.6)
+		(drill 0.3)
+		(layers "F.Cu" "B.Cu")
+		(net "BOOST_FB")
+	)
+	(segment
+		(start 87.6367 86.5316)
+		(end 87.6367 84.5144)
+		(width 0.18)
+		(layer "B.Cu")
+		(net "BOOST_FB")
+	)
+	(segment
+		(start 87.6367 84.5144)
+		(end 84.3755 81.2532)
+		(width 0.18)
+		(layer "B.Cu")
+		(net "BOOST_FB")
+	)
+	(segment
+		(start 81.5346 86.3167)
+		(end 81.5346 85.6271)
+		(width 0.18)
+		(layer "B.Cu")
+		(net "BOOST_FB")
+	)
+	(segment
+		(start 84.3755 81.2532)
+		(end 83.876 81.2532)
+		(width 0.18)
+		(layer "B.Cu")
+		(net "BOOST_FB")
+	)
+	(segment
+		(start 83.8625 88.6446)
+		(end 81.5346 86.3167)
+		(width 0.18)
+		(layer "B.Cu")
+		(net "BOOST_FB")
+	)
+	(segment
+		(start 83.8625 89.55)
+		(end 83.8625 88.6446)
+		(width 0.18)
+		(layer "B.Cu")
+		(net "BOOST_FB")
+	)
+	(segment
+		(start 83.876 81.2532)
+		(end 82.4762 82.653)
+		(width 0.18)
+		(layer "B.Cu")
+		(net "BOOST_FB")
 	)
 	(segment
